Commit message: modified

File: urdf/mobile_ur20.urdf (robot description, URDF)
Before this commit: robot ur20_robot, 11 links, 10 joints
Links:
- link base_link_inertia: geometry collision mesh filename=package://mobile_ur20_description/meshes/ur20/collision/bas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; visual mesh filename=package://mobile_ur20_description/meshes/ur20/visual/base.d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
- link forearm_link: geometry collision mesh filename=package://mobile_ur20_description/meshes/ur20/collision/for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; visual mesh filename=package://mobile_ur20_description/meshes/ur20/visual/forear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
- link shoulder_link: geometry collision mesh filename=package://mobile_ur20_description/meshes/ur20/collision/sho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; visual mesh filename=package://mobile_ur20_description/meshes/ur20/visual/should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
- link upper_arm_link: geometry collision mesh filename=package://mobile_ur20_description/meshes/ur20/collision/upp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; visual mesh filename=package://mobile_ur20_description/meshes/ur20/visual/uppera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
- link wrist_1_link: geometry collision mesh filename=package://mobile_ur20_description/meshes/ur20/collision/wri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; visual mesh filename=package://mobile_ur20_description/meshes/ur20/visual/wrist1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
- link wrist_2_link: geometry collision mesh filename=package://mobile_ur20_description/meshes/ur20/collision/wri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; visual mesh filename=package://mobile_ur20_description/meshes/ur20/visual/wrist2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
- link wrist_3_link: geometry collision mesh filename=package://mobile_ur20_description/meshes/ur20/collision/wri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; visual mesh filename=package://mobile_ur20_description/meshes/ur20/visual/wrist3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

File: urdf/obstacle.urdf (robot description, URDF)
Before this commit: robot obstacle, 1 links, 0 joints
Links:
- link obstacle_link: geometry collision box size=0.1 0.1 0.1; visual box size=0.1 0.1 0.1
